File: hardware/pcb/open_pocket.kicad_pcb (KiCad board)
At the start: 2 copper layers, 86 x 136 mm, 58 parts, among them J3 LCD 2.4in ILI9341, J4 LCD 1.44in ST7735 (alt.), J5 USB-C (charge), J6 LiPo 3.7 V, J7 Speaker 8R 1W, J8 3.5 mm, J9 Link port, Q1 BSS138, Q2 BSS138, Q3 BSS138, Q4 BSS138, Q5 AO3401, SW1 Up, SW10 Power, SW11 Wake / boost, SW2 Down, SW3 Left, SW4 Right, SW5 A, SW6 B, SW7 Select, SW8 Start, SW9 Menu, U1 Tang Nano 20K, U2 IP5306, U3 PAM8302A, U4 W25Q128JV

Commit message: Studio IDE with a board simulator; status icons; virtual printer; Menu pin
- apps/studio/sim: an RV32E interpreter runs the real fw.bin on a simulated board
  (iosys registers, W25Q flash and SD card at the SPI protocol level, OSD and LCD text,
  UART log, menu beeps, a FAT16 SD image built from a folder). Virtual time, so waits
  are skipped; sim/test_sim.js boots the firmware headless.
- Studio IDE tab: firmware sources in Monaco, Build (fw/build.sh), Run in the simulator,
  Flash to the board; HDMI and LCD menus drawn with the board's font, keyboard as the pad.
  The flash and SD images persist, so settings, saves and System Update can be tried.
  The Game Boy core itself is not emulated yet.
- Status icons in the menus: PC remote (a byte came over the UART), USB power (pin 86),
  battery level and charging from an IP5306-I2C on pins 15/16 (open drain).
- Tools > Virtual Printer: the core's serial port talks to the printer shifter inside the
  FPGA; pages go to /Prints and Tools > Last Print shows them on HDMI.
- Menu button of the carrier board on pin 54 (like S1).
- build.sh stops when every placer seed fails instead of packing an old placement.
  The bitstream with these RTL changes has not placed yet.
Parts:
- moved J3 73.0 mm to (179.5, 115.5)
- moved U1 18.0 mm to (127.6, 132.0)
